File: numpad/pcb/IC.sch (KiCad schematic (older format))
At the start: 5 parts, among them U3001 ATmega32U4-AU, Y3001 Crystal_GND24_Small

Commit message: updated all net label and connected the sheet pins
Parts:
- added R3001: 10K, symbol Device:R
- added SW3001: SW_Push, symbol Switch:SW_Push
Connections:
- net labels added: VCC, column_bus, row_bus, usb_d_N, usb_d_P
- net labels removed: 5v_post_fuse
- wire segments 31 -> 41
- no-connect marks 0 -> 18
Changed lines of the file:
@@
 $Descr A4 11693 8268
 encoding utf-8
-Sheet 3 5
+Sheet 2 4
 Title ""
 Date ""
@@
 $EndComp
 $Comp
-L power:GND #PWR03003
+L power:GND #PWR03004
 U 1 1 613B16A4
 P 7050 5800
-F 0 "#PWR03003" H 7050 5550 50  0001 C CNN
+F 0 "#PWR03004" H 7050 5550 50  0001 C CNN
 F 1 "GND" H 7055 5627 50  0000 C CNN
 F 2 "" H 7050 5800 50  0001 C CNN
@@
 Wire Wire Line
 	7050 5750 7050 5800
-Text GLabel 6400 2600 0    50   Input ~ 0
-IC_XTAL1
-Text GLabel 6400 2800 0    50   Input ~ 0
-IC_XTAL2
-Text Notes 6200 1600 0    157  ~ 0
-Microcontroller
 $Comp
 L Device:C C3003
@@
 	6250 3700 6250 3800
 $Comp
-L power:GND #PWR03002
+L power:GND #PWR03003
 U 1 1 613B16BA
 P 6250 4100
-F 0 "#PWR03002" H 6250 3850 50  0001 C CNN
+F 0 "#PWR03003" H 6250 3850 50  0001 C CNN
 F 1 "GND" H 6255 3927 50  0000 C CNN
 F 2 "" H 6250 4100 50  0001 C CNN
@@
 	4250 2450 4250 2150
 Connection ~ 4250 2450
-Text GLabel 3250 2150 1    50   Input ~ 0
-IC_XTAL1
-Text GLabel 4250 2150 1    50   Input ~ 0
-IC_XTAL2
 Wire Wire Line
 	3750 2250 3750 2350
@@
 Wire Wire Line
 	7050 1900 7150 1900
-Text GLabel 6850 1900 0    50   Input ~ 0
-5v_post_fuse
 Wire Wire Line
 	6400 2600 6550 2600
 Wire Wire Line
 	6400 2800 6550 2800
+Text HLabel 8050 2050 2    50   Input ~ 0
+row_bus
+Wire Bus Line
+	8050 2050 7850 2050
+Entry Wire Line
+	7750 2500 7850 2400
+Entry Wire Line
+	7750 2600 7850 2500
+Entry Wire Line
+	7750 2700 7850 2600
+Entry Wire Line
+	7750 2800 7850 2700
+Entry Wire Line
+	7750 2400 7850 2300
+Text HLabel 8050 3250 2    50   Output ~ 0
+column_bus
+Wire Bus Line
+	8050 3250 7850 3250
+Entry Wire Line
+	7750 3700 7850 3600
+Entry Wire Line
+	7750 3800 7850 3700
+Entry Wire Line
+	7750 3900 7850 3800
+Entry Wire Line
+	7750 3600 7850 3500
+NoConn ~ 7750 2900
+NoConn ~ 7750 3000
+NoConn ~ 7750 3100
+NoConn ~ 7750 3300
+NoConn ~ 7750 3400
+NoConn ~ 7750 4000
+NoConn ~ 7750 4100
+NoConn ~ 7750 4200
+NoConn ~ 7750 4300
+NoConn ~ 7750 4500
+NoConn ~ 7750 4600
+NoConn ~ 7750 4800
+NoConn ~ 7750 4900
+NoConn ~ 7750 5000
+NoConn ~ 7750 5100
+NoConn ~ 7750 5200
+NoConn ~ 7750 5300
+Text Label 6400 2600 2    50   ~ 0
+IC_XTAL1
+Text Label 6400 2800 2    50   ~ 0
+IC_XTAL2
+Text Label 3250 2150 2    50   ~ 0
+IC_XTAL1
+Text Label 4250 2150 0    50   ~ 0
+IC_XTAL2
+Text HLabel 6350 3200 0    50   Input ~ 0
+VCC
+Wire Wire Line
+	6350 3200 6550 3200
+Text HLabel 6350 3400 0    50   BiDi ~ 0
+usb_d_P
+Text HLabel 6350 3500 0    50   BiDi ~ 0
+usb_d_N
+Wire Wire Line
+	6350 3400 6550 3400
+Wire Wire Line
+	6350 3500 6550 3500
+NoConn ~ 6550 3000
+Text HLabel 5350 1950 0    50   Input ~ 0
+VCC
+$Comp
+L Device:R R3001
+U 1 1 613EDDBE
+P 5700 1950
+F 0 "R3001" V 5493 1950 50  0000 C CNN
+F 1 "10K" V 5584 1950 50  0000 C CNN
+F 2 "" V 5630 1950 50  0001 C CNN
+F 3 "~" H 5700 1950 50  0001 C CNN
+	1    5700 1950
+	0    1    1    0
+$EndComp
+Wire Wire Line
+	5350 1950 5550 1950
+Wire Wire Line
+	5850 1950 6150 1950
+Wire Wire Line
+	6150 2400 6550 2400
+$Comp
+L Switch:SW_Push SW3001
+U 1 1 613F2F7D
+P 5700 2400
+F 0 "SW3001" H 5700 2685 50  0000 C CNN
+F 1 "SW_Push" H 5700 2594 50  0000 C CNN
+F 2 "" H 5700 2600 50  0001 C CNN
+F 3 "~" H 5700 2600 50  0001 C CNN
+	1    5700 2400
+	1    0    0    -1
+$EndComp
+Wire Wire Line
+	6150 1950 6150 2400
+Wire Wire Line
+	6150 2400 5900 2400
+Connection ~ 6150 2400
+Wire Wire Line
+	5500 2400 5350 2400
+$Comp
+L power:GND #PWR03002
+U 1 1 613F79C7
+P 5350 2500
+F 0 "#PWR03002" H 5350 2250 50  0001 C CNN
+F 1 "GND" H 5355 2327 50  0000 C CNN
+F 2 "" H 5350 2500 50  0001 C CNN
+F 3 "" H 5350 2500 50  0001 C CNN
+	1    5350 2500
+	1    0    0    -1
+$EndComp
+Wire Wire Line
+	5350 2400 5350 2500
+Text HLabel 6850 1900 0    50   Input ~ 0
+VCC
+Text Notes 6200 1600 0    157  ~ 0
+Microcontroller
+Wire Bus Line
+	7850 3250 7850 3800
+Wire Bus Line
+	7850 2050 7850 2700
 $EndSCHEMATC
