File: numpad/pcb/power.sch (KiCad schematic (older format))
At the start: 5 parts

Commit message: updated all net label and connected the sheet pins
Parts:
- added F4001: 500m, symbol Device:Polyfuse_Small
- added J4001: USB_C_Receptacle_USB2.0, symbol numpad-rescue:USB_C_Receptacle_USB2.0-Connector
- renumbered C5001 to C4001, C5002 to C4002, C5003 to C4003, C5004 to C4004, C5005 to C4005
Connections:
- net labels added: usd_d_N, usd_d_P
- wire segments 21 -> 35
- no-connect marks 0 -> 4
Other:
- note added: "USB C 2.0"
Changed lines of the file:
@@
 $Descr A4 11693 8268
 encoding utf-8
-Sheet 5 5
+Sheet 3 4
 Title ""
 Date ""
@@
 $EndDescr
 $Comp
-L Device:C C5001
+L Device:C C4001
 U 1 1 613B5786
-P 2500 2600
-F 0 "C5001" H 2615 2646 50  0000 L CNN
-F 1 "0.1uF" H 2615 2555 50  0000 L CNN
-F 2 "" H 2538 2450 50  0001 C CNN
-F 3 "~" H 2500 2600 50  0001 C CNN
-	1    2500 2600
-	1    0    0    -1
-$EndComp
-Wire Wire Line
-	2500 2300 2500 2450
-$Comp
-L Device:C C5002
+P 2500 2450
+F 0 "C4001" H 2615 2496 50  0000 L CNN
+F 1 "0.1uF" H 2615 2405 50  0000 L CNN
+F 2 "" H 2538 2300 50  0001 C CNN
+F 3 "~" H 2500 2450 50  0001 C CNN
+	1    2500 2450
+	1    0    0    -1
+$EndComp
+Wire Wire Line
+	2500 2150 2500 2300
+$Comp
+L Device:C C4002
 U 1 1 613B578D
-P 3000 2600
-F 0 "C5002" H 3115 2646 50  0000 L CNN
-F 1 "0.1uF" H 3115 2555 50  0000 L CNN
-F 2 "" H 3038 2450 50  0001 C CNN
-F 3 "~" H 3000 2600 50  0001 C CNN
-	1    3000 2600
-	1    0    0    -1
-$EndComp
-Wire Wire Line
-	3000 2300 3000 2450
-$Comp
-L Device:C C5003
+P 3000 2450
+F 0 "C4002" H 3115 2496 50  0000 L CNN
+F 1 "0.1uF" H 3115 2405 50  0000 L CNN
+F 2 "" H 3038 2300 50  0001 C CNN
+F 3 "~" H 3000 2450 50  0001 C CNN
+	1    3000 2450
+	1    0    0    -1
+$EndComp
+Wire Wire Line
+	3000 2150 3000 2300
+$Comp
+L Device:C C4003
 U 1 1 613B5794
-P 3500 2600
-F 0 "C5003" H 3615 2646 50  0000 L CNN
-F 1 "0.1uF" H 3615 2555 50  0000 L CNN
-F 2 "" H 3538 2450 50  0001 C CNN
-F 3 "~" H 3500 2600 50  0001 C CNN
-	1    3500 2600
-	1    0    0    -1
-$EndComp
-Wire Wire Line
-	3500 2300 3500 2450
-$Comp
-L Device:C C5004
+P 3500 2450
+F 0 "C4003" H 3615 2496 50  0000 L CNN
+F 1 "0.1uF" H 3615 2405 50  0000 L CNN
+F 2 "" H 3538 2300 50  0001 C CNN
+F 3 "~" H 3500 2450 50  0001 C CNN
+	1    3500 2450
+	1    0    0    -1
+$EndComp
+Wire Wire Line
+	3500 2150 3500 2300
+$Comp
+L Device:C C4004
 U 1 1 613B579B
-P 4000 2600
-F 0 "C5004" H 4115 2646 50  0000 L CNN
-F 1 "0.1uF" H 4115 2555 50  0000 L CNN
-F 2 "" H 4038 2450 50  0001 C CNN
-F 3 "~" H 4000 2600 50  0001 C CNN
-	1    4000 2600
-	1    0    0    -1
-$EndComp
-Wire Wire Line
-	4000 2300 4000 2450
-$Comp
-L Device:C C5005
+P 4000 2450
+F 0 "C4004" H 4115 2496 50  0000 L CNN
+F 1 "0.1uF" H 4115 2405 50  0000 L CNN
+F 2 "" H 4038 2300 50  0001 C CNN
+F 3 "~" H 4000 2450 50  0001 C CNN
+	1    4000 2450
+	1    0    0    -1
+$EndComp
+Wire Wire Line
+	4000 2150 4000 2300
+$Comp
+L Device:C C4005
 U 1 1 613B57A2
-P 4500 2600
-F 0 "C5005" H 4615 2646 50  0000 L CNN
-F 1 "0.1uF" H 4615 2555 50  0000 L CNN
-F 2 "" H 4538 2450 50  0001 C CNN
-F 3 "~" H 4500 2600 50  0001 C CNN
-	1    4500 2600
-	1    0    0    -1
-$EndComp
-Wire Wire Line
-	4500 2300 4500 2450
-Wire Wire Line
-	2500 2300 3000 2300
-Connection ~ 3000 2300
-Wire Wire Line
-	3000 2300 3500 2300
-Connection ~ 3500 2300
-Wire Wire Line
-	3500 2300 4000 2300
-Connection ~ 4000 2300
-Wire Wire Line
-	4000 2300 4500 2300
-Wire Wire Line
-	2500 2750 2500 2900
-Wire Wire Line
-	3000 2750 3000 2900
-Wire Wire Line
-	4000 2750 4000 2900
-Wire Wire Line
-	4500 2750 4500 2900
-Wire Wire Line
-	4500 2900 4000 2900
-Connection ~ 3000 2900
-Wire Wire Line
-	3000 2900 2500 2900
-Connection ~ 3500 2900
-Wire Wire Line
-	3500 2900 3000 2900
-Connection ~ 4000 2900
-Wire Wire Line
-	4000 2900 3500 2900
-Text GLabel 3450 2050 0    50   Input ~ 0
+P 4500 2450
+F 0 "C4005" H 4615 2496 50  0000 L CNN
+F 1 "0.1uF" H 4615 2405 50  0000 L CNN
+F 2 "" H 4538 2300 50  0001 C CNN
+F 3 "~" H 4500 2450 50  0001 C CNN
+	1    4500 2450
+	1    0    0    -1
+$EndComp
+Wire Wire Line
+	4500 2150 4500 2300
+Wire Wire Line
+	2500 2150 3000 2150
+Connection ~ 3000 2150
+Wire Wire Line
+	3000 2150 3500 2150
+Connection ~ 3500 2150
+Wire Wire Line
+	3500 2150 4000 2150
+Connection ~ 4000 2150
+Wire Wire Line
+	4000 2150 4500 2150
+Wire Wire Line
+	2500 2600 2500 2750
+Wire Wire Line
+	3000 2600 3000 2750
+Wire Wire Line
+	4000 2600 4000 2750
+Wire Wire Line
+	4500 2600 4500 2750
+Wire Wire Line
+	4500 2750 4000 2750
+Connection ~ 3000 2750
+Wire Wire Line
+	3000 2750 2500 2750
+Connection ~ 3500 2750
+Wire Wire Line
+	3500 2750 3000 2750
+Connection ~ 4000 2750
+Wire Wire Line
+	4000 2750 3500 2750
+Wire Wire Line
+	3500 1900 3500 2150
+$Comp
+L power:GND #PWR04001
+U 1 1 613B57BE
+P 3500 2900
+F 0 "#PWR04001" H 3500 2650 50  0001 C CNN
+F 1 "GND" H 3505 2727 50  0000 C CNN
+F 2 "" H 3500 2900 50  0001 C CNN
+F 3 "" H 3500 2900 50  0001 C CNN
+	1    3500 2900
+	1    0    0    -1
+$EndComp
+Wire Wire Line
+	3500 2600 3500 2750
+Wire Wire Line
+	3500 2750 3500 2900
+Text Notes 2400 1650 0    157  ~ 0
+Decoupling Resistor
+$Comp
+L numpad-rescue:USB_C_Receptacle_USB2.0-Connector J?
+U 1 1 6138A3A7
+P 6350 2900
+AR Path="/613893FD/6138A3A7" Ref="J?"  Part="1"
+AR Path="/613B1F02/6138A3A7" Ref="J4001"  Part="1"
+F 0 "J4001" H 6457 3767 50  0000 C CNN
+F 1 "USB_C_Receptacle_USB2.0" H 6457 3676 50  0000 C CNN
+F 2 "" H 6500 2900 50  0001 C CNN
+F 3 "https://www.usb.org/sites/default/files/documents/usb_type-c.zip" H 6500 2900 50  0001 C CNN
+	1    6350 2900
+	1    0    0    -1
+$EndComp
+Text Notes 6350 1750 0    157  ~ 0
+USB C 2.0
+Wire Wire Line
+	6950 2800 7100 2800
+Wire Wire Line
+	7100 2800 7100 2900
+Wire Wire Line
+	6950 2900 7100 2900
+Wire Wire Line
+	6950 3000 7100 3000
+Wire Wire Line
+	7100 3000 7100 3100
+Wire Wire Line
+	6950 3100 7100 3100
+$Comp
+L Device:Polyfuse_Small F?
+U 1 1 6138A3B6
+P 7300 2300
+AR Path="/613893FD/6138A3B6" Ref="F?"  Part="1"
+AR Path="/613B1F02/6138A3B6" Ref="F4001"  Part="1"
+F 0 "F4001" V 7095 2300 50  0000 C CNN
+F 1 "500m" V 7186 2300 50  0000 C CNN
+F 2 "" H 7350 2100 50  0001 L CNN
+F 3 "~" H 7300 2300 50  0001 C CNN
+	1    7300 2300
+	0    1    1    0
+$EndComp
+Wire Wire Line
+	7100 3100 7700 3100
+Connection ~ 7100 3100
+NoConn ~ 6950 3400
+NoConn ~ 6950 3500
+$Comp
+L power:GND #PWR?
+U 1 1 6138A3C4
+P 6350 4100
+AR Path="/613893FD/6138A3C4" Ref="#PWR?"  Part="1"
+AR Path="/613B1F02/6138A3C4" Ref="#PWR04002"  Part="1"
+F 0 "#PWR04002" H 6350 3850 50  0001 C CNN
+F 1 "GND" H 6355 3927 50  0000 C CNN
+F 2 "" H 6350 4100 50  0001 C CNN
+F 3 "" H 6350 4100 50  0001 C CNN
+	1    6350 4100
+	1    0    0    -1
+$EndComp
+Wire Wire Line
+	6050 3800 6050 3950
+Wire Wire Line
+	6050 3950 6350 3950
+Wire Wire Line
+	6350 3950 6350 3800
+Wire Wire Line
+	6350 3950 6350 4100
+Connection ~ 6350 3950
+Text HLabel 7700 2300 2    50   Output ~ 0
 5v_post_fuse
 Wire Wire Line
-	3450 2050 3500 2050
-Wire Wire Line
-	3500 2050 3500 2300
-$Comp
-L power:GND #PWR05001
-U 1 1 613B57BE
-P 3500 3050
-F 0 "#PWR05001" H 3500 2800 50  0001 C CNN
-F 1 "GND" H 3505 2877 50  0000 C CNN
-F 2 "" H 3500 3050 50  0001 C CNN
-F 3 "" H 3500 3050 50  0001 C CNN
-	1    3500 3050
-	1    0    0    -1
-$EndComp
-Wire Wire Line
-	3500 2750 3500 2900
-Wire Wire Line
-	3500 2900 3500 3050
-Text Notes 2400 1800 0    157  ~ 0
-Decoupling Resistor
+	6950 2300 7200 2300
+Text HLabel 7700 2900 2    50   BiDi ~ 0
+usd_d_N
+Connection ~ 7100 2900
+Wire Wire Line
+	7100 2900 7700 2900
+Text HLabel 7700 3100 2    50   BiDi ~ 0
+usd_d_P
+NoConn ~ 6950 2500
+NoConn ~ 6950 2600
+Wire Wire Line
+	7400 2300 7700 2300
+Text HLabel 3400 1900 0    50   Input ~ 0
+5v_post_fuse
+Wire Wire Line
+	3400 1900 3500 1900
 $EndSCHEMATC
